File: Electronic/Schematic/RollerShutterController/RollerShutterController.kicad_sch (KiCad schematic)
At the start: 6 parts, among them U1 LDK320M33R

Commit message: Added electronic project.
Signed-off-by: Kamil Lazowski <autobrewing@gmail.com>
Parts:
- added JP1: SolderJumper_2_Bridged, Jumper:SolderJumper-2_P1.3mm_Bridged_Pad1.0x1.5mm, symbol Jumper:SolderJumper_2_Bridged
- C1, C2: value 1u -> 1u 25V; footprint (none) -> Capacitor_SMD:C_0603_1608Metric_Pad1.08x0.95mm_HandSolder
- D1: footprint Diode_SMD:D_SOD-323 -> Diode_SMD:D_SOD-323_HandSoldering
- D2: footprint Diode_SMD:D_SOD-323F -> Diode_SMD:D_SOD-323_HandSoldering
Connections:
- net GND: now also JP1.2 (B); no longer C2.2, D2.2 (A), U1.2 (GND)
- net +12V_SAFE: now reaches C2.1, D2.1 (K), F1.2, U1.1 (IN), U1.3 (EN)
- net +3.3V renamed +3V3
- new net GNDPWR: C2.2, D2.2 (A), JP1.1 (A), U1.2 (GND)
