File: Electronic/Schematic/RollerShutterController/connectors.kicad_sch (KiCad schematic)
At the start: 4 parts, among them J1 Conn_01x02_Socket, J2 Conn_01x02_Socket, J3 Conn_01x02_Socket, J4 Conn_01x03_Socket

Commit message: Added electronic project.
Signed-off-by: Kamil Lazowski <autobrewing@gmail.com>
Parts:
- removed J3: Conn_01x02_Socket, symbol Connector:Conn_01x02_Socket
- added J6: Conn_01x03_Socket, TerminalBlock:TerminalBlock_Xinya_XY308-2.54-3P_1x03_P2.54mm_Horizontal, symbol Connector:Conn_01x03_Socket
- J1: footprint Connector_RJ:RJ45_Pulse_JK0654219NL_Horizontal -> TerminalBlock:TerminalBlock_Xinya_XY308-2.54-2P_1x02_P2.54mm_Horizontal
- J2: footprint (none) -> TerminalBlock:TerminalBlock_Xinya_XY308-2.54-2P_1x02_P2.54mm_Horizontal
- J4: footprint (none) -> DG301-5.0:DG301-5.0
Connections:
- net 230V AC is gone; now on net MOTOR_DOWN: J4.2 (Pin_2)
- net BUTTON_LOCAL_DOWN_EXT: now also J6.1 (Pin_1)
- net BUTTON_LOCAL_UP_EXT: now also J6.3 (Pin_3)
- net BUTTON_REMOTE_DOWN_EXT: now also J2.1 (Pin_1); no longer J2.2 (Pin_2)
- net BUTTON_REMOTE_UP_EXT: now also J2.2 (Pin_2); no longer J2.1 (Pin_1)
- net MOTOR_DOWN: no longer J4.3 (Pin_3)
- net +12 VDC renamed GNDPWR
- net GNDPWR: now also J6.2 (Pin_2)
- net 0 VDC renamed +12V
- new net 230V_AC: J4.3 (Pin_3)
Other:
- moved on the sheet: J1
