File: Electronic/Schematic/RollerShutterController/mcu.kicad_sch (KiCad schematic)
At the start: 3 parts, among them U2 STM32C011F4Px

Commit message: Added electronic project.
Signed-off-by: Kamil Lazowski <autobrewing@gmail.com>
Parts:
- added J3: TC2030, Connector:Tag-Connect_TC2030-IDC-NL_2x03_P1.27mm_Vertical, symbol Connector:TC2030
- C3: value 100n -> 100n 50V; footprint (none) -> Capacitor_SMD:C_0603_1608Metric_Pad1.08x0.95mm_HandSolder
- C4: value 4,7u -> 1u 25V; footprint (none) -> Capacitor_SMD:C_0603_1608Metric_Pad1.08x0.95mm_HandSolder
Connections:
- net +3V3: now also J3.1
- net GND: now also J3.5
- net RELAY_UP: now reaches U2.1 (PB7)
- net BUTTON_LOCAL_DOWN: now reaches U2.11 (PA4)
- net BUTTON_LOCAL_UP: now reaches U2.15 (PA8)
- net BUTTON_REMOTE_DOWN: now reaches U2.16 (PA9/PA11)
- net BUTTON_REMOTE_UP: now reaches U2.17 (PA10/PA12)
- net SWDIO: now reaches U2.18 (PA13)
- net SWDIO: now also J3.2
- net SWCLK: now reaches U2.19 (PA14)
- net SWCLK: now also J3.4
- net RELAY_DOWN: now reaches U2.2 (PC14)
- net BUZZER: now reaches U2.3 (PC15)
- net NRST: now reaches U2.6 (PF2)
- net NRST: now also J3.3
- no-connect marks 0 -> 9
Other:
- note added: "Debugger connector TC2030 Connector"
- moved on the sheet: C3
