File: Electronic/Schematic/RollerShutterController/relay.kicad_sch (KiCad schematic)
At the start: 10 parts, among them K1 AZ921-1A-12DE, K2 AZ921-1A-12DE, Q1 BSS138, Q2 BSS138

Commit message: Added electronic project.
Signed-off-by: Kamil Lazowski <autobrewing@gmail.com>
Parts:
- D3, D4: footprint Diode_SMD:D_SOD-323 -> Diode_SMD:D_SOD-323_HandSoldering
- K1, K2: footprint Package_DIP:DIP-8_W7.62mm -> AZ921:AZ921
- R1, R4: footprint Diode_SMD:D_SOD-323 -> Resistor_SMD:R_0603_1608Metric_Pad0.98x0.95mm_HandSolder
- R2, R3: footprint (none) -> Resistor_SMD:R_0603_1608Metric_Pad0.98x0.95mm_HandSolder
Connections:
- net MOTOR_DOWN: now also K2.14; no longer K2.13
- net MOTOR_UP: now also K1.14; no longer K1.13
- net at D4.2 (A), Q2.3 (D): now also K2.A1; no longer K2.A2
- net at D3.2 (A), Q1.3 (D): now also K1.A1; no longer K1.A2
- net +12V renamed +12V_SAFE
- net +12V_SAFE: now also K1.A2, K2.A2; no longer K1.A1, K2.A1
- removed net 230V AC: K1.14, K2.14
- net GND renamed GNDPWR
- new net 230V_AC: K1.13, K2.13
