File: Electronic/Schematic/RollerShutterController/RollerShutterController.kicad_pcb (KiCad board)
At the start: 2 copper layers, 40 x 37 mm, 47 parts, among them J1 Conn_01x02_Socket, J2 Conn_01x02_Socket, J3 TC2030, J4 Conn_01x03_Socket, J6 Conn_01x03_Socket, K1 AZ921-1A-12DE, K2 AZ921-1A-12DE, Q1 BSS138, Q2 BSS138, Q3 BSS138, U1 LDK320M33R, U2 STM32C011F4Px, U4 LTV-247

Commit message: Added PCB production files.
Signed-off-by: Kamil Lazowski <autobrewing@gmail.com>
Parts:
- moved J1 1.62 mm to (176.2, 65.9)
- moved J2 1.40 mm to (182.9, 65.9)
- moved J6 1.40 mm to (192.1, 65.9)
- moved J4 0.86 mm to (161.4, 69.6)
Routing:
- net GND: track 15.5 -> 17.0 mm, vias 34 -> 36
- net MOTOR_UP: track 14.4 -> 13.5 mm, vias 5 -> 4
- net 230V_AC: track 43.8 -> 42.9 mm
- net BUTTON_LOCAL_DOWN_EXT: track 8.41 -> 7.83 mm
- net BUTTON_REMOTE_DOWN_EXT: track 8.26 -> 7.68 mm
- net BUTTON_LOCAL_UP_EXT: track 8.84 -> 8.26 mm
- net BUTTON_REMOTE_UP_EXT: track 7.65 -> 7.07 mm
- net +12V: track 51.8 -> 51.2 mm
Other:
- board size 40 x 37 mm -> 41 x 38 mm
